File: hardware/MCU_INTERFACE_BOARD/MCU_INTERFACE_BOARD.sch (KiCad schematic (older format))
At the start: 4 parts, among them J1 IDC_02x04, J2 IDC_02x04, J4 Conn_01x10, J5\ Conn_01x10

Commit message: Finish development
Parts:
- added D1: LED, LED_SMD:LED_0805_2012Metric, symbol Device:LED
- added J3: Conn_02x10_Odd_Even, Connector_IDC:IDC-Header_2x10_P2.54mm_Vertical, symbol Connector_Generic:Conn_02x10_Odd_Even
- added J6: Screw_Terminal_01x02, TerminalBlock_4Ucon:TerminalBlock_4Ucon_1x02_P3.50mm_Horizontal, symbol Connector:Screw_Terminal_01x02
- added R1: 220, Resistor_THT:R_Axial_DIN0207_L6.3mm_D2.5mm_P10.16mm_Horizontal, symbol Device:R
- added R2, R3: 4.7K, Resistor_THT:R_Axial_DIN0207_L6.3mm_D2.5mm_P10.16mm_Horizontal, symbol Device:R
- J1, J2: footprint (none) -> Connector_IDC:IDC-Header_2x04_P2.54mm_Vertical
- J4: footprint (none) -> Connector_PinHeader_2.54mm:PinHeader_1x10_P2.54mm_Vertical
- J5: renamed from J5\; footprint (none) -> Connector_PinHeader_2.54mm:PinHeader_1x10_P2.54mm_Vertical
Connections:
- net PULL is gone; now on net +5V: J1.3 (Pin_3), J2.3 (Pin_3)
- net PUSH is gone; now on net GND: J1.4 (Pin_4), J2.4 (Pin_4)
- net GND: now also J4.3 (Pin_3), D1.1 (K), J3.5 (Pin_5), J6.2 (Pin_2)
- net SCL: now also J3.7 (Pin_7), R3.2
- net SDA: now also J3.9 (Pin_9), R2.2
- net VCC: now also J4.2 (Pin_2), J3.3 (Pin_3), R2.1, R3.1
- net +5V: now reaches J4.1 (Pin_1)
- net +5V: now also J3.1 (Pin_1), J6.1 (Pin_1), R1.2
- net GPIO5: now reaches J4.10 (Pin_10)
- net GPIO5: now also J3.4 (Pin_4)
- net ESP_EN: now reaches J4.4 (Pin_4)
- net ESP_EN: now also J3.11 (Pin_11)
- net GPIO0: now reaches J4.5 (Pin_5)
- net GPIO0: now also J3.13 (Pin_13)
- net GPIO1: now reaches J4.6 (Pin_6)
- net GPIO1: now also J3.15 (Pin_15)
- net GPIO2: now reaches J4.7 (Pin_7)
- net GPIO2: now also J3.17 (Pin_17)
- net GPIO3: now reaches J4.8 (Pin_8)
- net GPIO3: now also J3.19 (Pin_19)
- net GPIO4: now reaches J4.9 (Pin_9)
- net GPIO4: now also J3.2 (Pin_2)
- net GPI39: now reaches J5.1 (Pin_1)
- net GPI39: now also J3.6 (Pin_6)
- net GPIO13: now reaches J5.10 (Pin_10)
- net GPIO13: now also J3.20 (Pin_20)
- net GPI36: now reaches J5.2 (Pin_2)
- net GPI36: now also J3.8 (Pin_8)
- net GPI35: now reaches J5.3 (Pin_3)
- net GPI35: now also J3.10 (Pin_10)
- net GPI34: now reaches J5.4 (Pin_4)
- net GPI34: now also J3.12 (Pin_12)
- net GPIO16: now reaches J5.7 (Pin_7)
- net GPIO16: now also J3.14 (Pin_14)
- net GPIO15: now reaches J5.8 (Pin_8)
- net GPIO15: now also J3.16 (Pin_16)
- net GPIO14: now reaches J5.9 (Pin_9)
- net GPIO14: now also J3.18 (Pin_18)
- new net: D1.2 (A), R1.1
- no-connect marks 1 -> 0
Other:
- note added: "5V input"
- note added: "BUS connectors"
- note added: "BUS pullups"
- note added: "GPIO connector"
- note added: "OLIMEX ESP32-POE socket"
- note added: "PUSH&PULL to\npower"
- note added: "Power LED"
- moved on the sheet: J1, J2, J4, J5
