File: hardware/SWITCH_INPUT_BOARD/SWITCH_INPUT_BOARD.kicad_pcb (KiCad board)
At the start: 2 copper layers, 82.2 x 67.2 mm, 37 parts, among them J1 4 Port RJ45: A00-432-262-450, J2 IDC_02x04, J3 IDC_02x04, J4 IDC_02x04, J5 IDC_02x06, U1 MCP23017_SO

Commit message: Finish development
Other:
- net class Default removed
- board text added: "1 2"
- board text added: "10K"
- board text added: "10uF"
- board text added: "1: PUSH->GND"
- board text added: "1K"
- board text added: "220"
- board text added: "2: PULL->VCC"
- board text added: "4.7K"
- board text added: "JLCJLCJLCJLC"
- board text removed: "JP4: PULL->VCC"
- board text removed: "JP5: PUSH->GND"
