File: hardware/TERMINATOR_BOARD/TERMINATOR_BOARD.kicad_pcb (KiCad board)
At the start: 2 copper layers, 22 x 48 mm, 4 parts, among them J1 *, J2 *

Commit message: Finish development
Other:
- net class Default removed
- board text added: "JLCJLCJLCJLC"
